File: OBC2.kicad_pcb (KiCad board)
At the start: 2 copper layers, 95.9 x 90.2 mm, 81 parts, among them IC1 LTC4411, IC2 LTC4411, J1 Conn_02x30_Row_Letter_First, J2 Conn_02x30_Row_Letter_First, J3 USB_B, J4 8P8C_Shielded, J5 Conn_02x07_Odd_Even, U1 USBLC6-2SC6, U2 R-783.3-0.5, U3 STM32F407VETx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

Commit message: correct flipped i2c1 SCL SDA lines
Parts:
- J5: value Conn_02x07_Odd_Even -> FTSH-107-01-F-DV-K
- U5: footprint Package_SO:SOIC-8_5.23x5.23mm_P1.27mm -> Package_SO:SOIC-8_5.3x5.3mm_P1.27mm
Connections:
- J1 pad a20: /I2C1_SDA -> /I2C1_SCL
- J1 pad b20: /I2C1_SCL -> /I2C1_SDA
- R4 pad 1: /I2C1_SDA -> /I2C1_SCL
- R5 pad 1: /I2C1_SCL -> /I2C1_SDA
- U3 pad 92: /I2C1_SDA -> /I2C1_SCL
- U3 pad 93: /I2C1_SCL -> /I2C1_SDA
Routing:
- net /I2C1_SDA: track 89.4 -> 90.3 mm
- net /I2C1_SCL: track 90.3 -> 89.4 mm
